File: MOTOR_DRIVER_PCB/PCB_24V_CONVERT/PCB_24V_CONVERT.kicad_pcb (KiCad board)
At the start: 2 copper layers, 212 x 192 mm, 49 parts, among them J1 BATT_24V_IN, J10 ARDUINO2_5V, J2 MAIN_SW_LOWI, J3 MDD10A_1, J4 MDD10A_2, J5 STEPPER_24V, J6 SERVO_12V, J7 JETSON_19V, J8 ARDUINO_5V, J9 CTRL_SENSE, K1 CONTACTOR_24V, K2 RELAY_BYPASS, Q1 2N7002, U1 XL4016_12V, U2 BUCK_19V_DNP, U3 BUCK_5V

Commit message: 팔 구동 펌웨어(Herkulex/스테퍼) + PCB 업데이트
- Herkulex DRS-0601 제어(herkulex_0601_control): setid로 ID부여/scan/각도측정, 진단(stat/ack/loop), 빠른 스캔(12ms)
- 스테퍼 ST-NK1748E 제어/테스트(urt/arm_stepper_control, arm_stepper_test)
- Herkulex 원시 프로토콜 파이썬 테스트(tests/herkulex_test.py)
- MOTOR_DRIVER_PCB: MEGA_SHIELD 프로젝트/24V 컨버터 업데이트 + 산출물(exports)
- CP210x Windows 드라이버 동봉

Co-Authored-By: Claude Opus 4.8 <noreply@anthropic.com>
Parts:
- added J11: FAN1_5V, TerminalBlock_Phoenix:TerminalBlock_Phoenix_MKDS-3-2-5.08_1x02_P5.08mm_Horizontal, F.Cu at (105.0, 165.0)
- added J12: FAN2_5V, TerminalBlock_Phoenix:TerminalBlock_Phoenix_MKDS-3-2-5.08_1x02_P5.08mm_Horizontal, F.Cu at (128.0, 165.0)
Connections:
- net /GND renamed GND
- net /V24 renamed +24V
Routing:
- net /V5: track 234.7 -> 295.7 mm
