File: MOTOR_DRIVER_PCB/PCB_24V_CONVERT/PCB_24V_CONVERT.kicad_sch (KiCad schematic)
At the start: 0 parts

Commit message: MOTOR_DRIVER_PCB: 24V 컨버터 PCB 업데이트 + 전원 가이드/산출물
- PCB_24V_CONVERT (kicad pcb/sch/pro/prl) 갱신 + PCB_24V_CONVERT_MIN 변형 추가
- KICAD_POWER_GUIDE.md, exports/(schematic/pcb PDF·SVG·PNG·BOM 문서)
- DRC/ERC 리포트(PCB_24V_CONVERT, _MIN), radio_schematic(schematic.html)

Co-Authored-By: Claude Opus 4.8 <noreply@anthropic.com>
Parts:
- added C1: 1000uF/50V, Capacitor_THT:CP_Radial_D12.5mm_P5.00mm, symbol Device:C_Polarized
- added C10, C6: 0.1uF/50V, Capacitor_THT:C_Disc_D5.0mm_W2.5mm_P5.00mm, symbol Device:C
- added C2: 470uF/50V, Capacitor_THT:CP_Radial_D10.0mm_P5.00mm, symbol Device:C_Polarized
- added C3: 1000uF/25V, Capacitor_THT:CP_Radial_D10.0mm_P5.00mm, symbol Device:C_Polarized
- added C4: 470uF/16V, Capacitor_THT:CP_Radial_D8.0mm_P3.50mm, symbol Device:C_Polarized
- added C5: 470uF/35V, Capacitor_THT:CP_Radial_D10.0mm_P5.00mm, symbol Device:C_Polarized
- added C7, C8: 0.1uF/25V, Capacitor_THT:C_Disc_D5.0mm_W2.5mm_P5.00mm, symbol Device:C
- added C9: 0.1uF/16V, Capacitor_THT:C_Disc_D5.0mm_W2.5mm_P5.00mm, symbol Device:C
- added D1: SMBJ13A, Diode_SMD:D_SMB, symbol Device:D_TVS
- added D2: SMBJ30A, Diode_SMD:D_SMB, symbol Device:D_TVS
- added D3: SMBJ6.0A, Diode_SMD:D_SMB, symbol Device:D_TVS
- added D4: SMBJ20A, Diode_SMD:D_SMB, symbol Device:D_TVS
- added D5: FLYBACK_K1, Diode_THT:D_DO-41_SOD81_P7.62mm_Horizontal, symbol Device:D
- added D6: FLYBACK_K2, Diode_THT:D_DO-41_SOD81_P7.62mm_Horizontal, symbol Device:D
- added F1: 25A_MAIN, Fuse:FuseHolder_Blade_ATO_Littelfuse_FLR_178.6165, symbol Device:Fuse
- added F2, F3: 15A, Fuse:FuseHolder_Blade_ATO_Littelfuse_FLR_178.6165, symbol Device:Fuse
- added F4, F8: 10A, Fuse:FuseHolder_Blade_ATO_Littelfuse_FLR_178.6165, symbol Device:Fuse
- added F5: 7.5A, Fuse:FuseHolder_Blade_ATO_Littelfuse_FLR_178.6165, symbol Device:Fuse
- added F6: 5A, Fuse:FuseHolder_Blade_ATO_Littelfuse_FLR_178.6165, symbol Device:Fuse
- added F7: 2A, Fuse:FuseHolder_Blade_ATO_Littelfuse_FLR_178.6165, symbol Device:Fuse
- added J1: BATT_24V_IN, Connector_AMASS:AMASS_XT60PW-M_1x02_P7.20mm_Horizontal, symbol Connector_Generic:Conn_01x02
- added J10: ARDUINO2_5V, TerminalBlock_Phoenix:TerminalBlock_Phoenix_MKDS-3-2-5.08_1x02_P5.08mm_Horizontal, symbol Connector_Generic:Conn_01x02
- added J2: MAIN_SW_LOWI, TerminalBlock_Phoenix:TerminalBlock_Phoenix_MKDS-3-2-5.08_1x02_P5.08mm_Horizontal, symbol Connector_Generic:Conn_01x02
- added J3: MDD10A_1, TerminalBlock_Phoenix:TerminalBlock_Phoenix_MKDS-3-2-5.08_1x02_P5.08mm_Horizontal, symbol Connector_Generic:Conn_01x02
- added J4: MDD10A_2, TerminalBlock_Phoenix:TerminalBlock_Phoenix_MKDS-3-2-5.08_1x02_P5.08mm_Horizontal, symbol Connector_Generic:Conn_01x02
- added J5: STEPPER_24V, TerminalBlock_Phoenix:TerminalBlock_Phoenix_MKDS-3-2-5.08_1x02_P5.08mm_Horizontal, symbol Connector_Generic:Conn_01x02
- added J6: SERVO_12V, TerminalBlock_Phoenix:TerminalBlock_Phoenix_MKDS-3-2-5.08_1x02_P5.08mm_Horizontal, symbol Connector_Generic:Conn_01x02
- added J7: JETSON_19V, TerminalBlock_Phoenix:TerminalBlock_Phoenix_MKDS-3-2-5.08_1x02_P5.08mm_Horizontal, symbol Connector_Generic:Conn_01x02
- added J8: ARDUINO_5V, TerminalBlock_Phoenix:TerminalBlock_Phoenix_MKDS-3-2-5.08_1x02_P5.08mm_Horizontal, symbol Connector_Generic:Conn_01x02
- added J9: CTRL_SENSE, Connector_PinHeader_2.54mm:PinHeader_1x03_P2.54mm_Vertical, symbol Connector_Generic:Conn_01x03
- added K1: CONTACTOR_24V, TerminalBlock_Phoenix:TerminalBlock_Phoenix_MKDS-3-4-5.08_1x04_P5.08mm_Horizontal, symbol Connector_Generic:Conn_01x04
- added K2: RELAY_BYPASS, TerminalBlock_Phoenix:TerminalBlock_Phoenix_MKDS-3-4-5.08_1x04_P5.08mm_Horizontal, symbol Connector_Generic:Conn_01x04
- added Q1: 2N7002, Package_TO_SOT_SMD:SOT-23, symbol Transistor_FET:2N7002
- added R1: 120k, Resistor_THT:R_Axial_DIN0207_L6.3mm_D2.5mm_P7.62mm_Horizontal, symbol Device:R
- added R2: 22k, Resistor_THT:R_Axial_DIN0207_L6.3mm_D2.5mm_P7.62mm_Horizontal, symbol Device:R
- added R3: 100R, Resistor_THT:R_Axial_DIN0207_L6.3mm_D2.5mm_P7.62mm_Horizontal, symbol Device:R
- added R4: 100k, Resistor_THT:R_Axial_DIN0207_L6.3mm_D2.5mm_P7.62mm_Horizontal, symbol Device:R
- added RT1: NTC_2R_25A, Varistor:RV_Disc_D12mm_W5.8mm_P7.5mm, symbol Device:Thermistor
- added U1: XL4016_12V, TerminalBlock_Phoenix:TerminalBlock_Phoenix_MKDS-3-4-5.08_1x04_P5.08mm_Horizontal, symbol Connector_Generic:Conn_01x04
- added U2: BUCK_19V_DNP, TerminalBlock_Phoenix:TerminalBlock_Phoenix_MKDS-3-4-5.08_1x04_P5.08mm_Horizontal, symbol Connector_Generic:Conn_01x04
- added U3: BUCK_5V, TerminalBlock_Phoenix:TerminalBlock_Phoenix_MKDS-3-4-5.08_1x04_P5.08mm_Horizontal, symbol Connector_Generic:Conn_01x04
Connections:
- new net BATT+: F1.1, J1.1 (Pin_1)
- new net BK12_IN: C2.1, F5.2, U1.1 (Pin_1)
- new net BK19_IN: F6.2, U2.1 (Pin_1)
- new net BK5_IN: F7.2, U3.1 (Pin_1)
- new net FUSED: F1.2, J2.1 (Pin_1), K1.1 (Pin_1)
- new net GND: C1.2, C10.2, C2.2, C3.2, C4.2, C5.2, C6.2, C7.2, C8.2, C9.2, D1.2 (A2), D2.2 (A2), D3.2 (A2), D4.2 (A2), D5.2 (A), J1.2 (Pin_2), J10.2 (Pin_2), J3.2 (Pin_2), J4.2 (Pin_2), J5.2 (Pin_2), J6.2 (Pin_2), J7.2 (Pin_2), J8.2 (Pin_2), J9.3 (Pin_3), K1.4 (Pin_4), Q1.2 (S), R2.2, R4.2, U1.2 (Pin_2), U1.4 (Pin_4), U2.2 (Pin_2), U2.4 (Pin_4), U3.2 (Pin_2), U3.4 (Pin_4)
- new net K1_COIL: D5.1 (K), J2.2 (Pin_2), K1.3 (Pin_3)
- new net K2_DRV: J9.1 (Pin_1), R3.1
- new net K2_GATE: Q1.1 (G), R3.2, R4.1
- new net K2_LS: D6.2 (A), K2.4 (Pin_4), Q1.3 (D)
- new net MDD1_F: F2.2, J3.1 (Pin_1)
- new net MDD2_F: F3.2, J4.1 (Pin_1)
- new net STEP_F: F4.2, J5.1 (Pin_1)
- new net SW_MAIN: D6.1 (K), K1.2 (Pin_2), K2.1 (Pin_1), K2.3 (Pin_3), RT1.1
- new net V12: C3.1, F8.1, U1.3 (Pin_3)
- new net V12_OUT: C7.1, D1.1 (A1), F8.2, J6.1 (Pin_1)
- new net V19: C5.1, C8.1, D4.1 (A1), J7.1 (Pin_1), U2.3 (Pin_3)
- new net V24: C1.1, C6.1, D2.1 (A1), F2.1, F3.1, F4.1, F5.1, F6.1, F7.1, K2.2 (Pin_2), R1.1, RT1.2
- new net V5: C4.1, C9.1, D3.1 (A1), J10.1 (Pin_1), J8.1 (Pin_1), U3.3 (Pin_3)
- new net VBAT_SENSE: C10.1, J9.2 (Pin_2), R1.2, R2.1
Other:
- note added: "K1 contactor: J2 low-current switch drives coil + D5 flyback. K2 bypass: Q1(2N7002 low-side)+Rg/Rgs gate+D6 flyback; MCU drives gate ~500ms after inrush via J9(CTRL). Bucks U1/U2/U3 EN=always-on(verify pullup), U2=DNP. U4/K1/K2 need real part numbers. Provisional F1(BMS)/F4(stepper)/servo-stall/7S."

Commit message: 팔 구동 펌웨어(Herkulex/스테퍼) + PCB 업데이트
- Herkulex DRS-0601 제어(herkulex_0601_control): setid로 ID부여/scan/각도측정, 진단(stat/ack/loop), 빠른 스캔(12ms)
- 스테퍼 ST-NK1748E 제어/테스트(urt/arm_stepper_control, arm_stepper_test)
- Herkulex 원시 프로토콜 파이썬 테스트(tests/herkulex_test.py)
- MOTOR_DRIVER_PCB: MEGA_SHIELD 프로젝트/24V 컨버터 업데이트 + 산출물(exports)
- CP210x Windows 드라이버 동봉

Co-Authored-By: Claude Opus 4.8 <noreply@anthropic.com>
Parts:
- added J11: FAN1_5V, TerminalBlock_Phoenix:TerminalBlock_Phoenix_MKDS-3-2-5.08_1x02_P5.08mm_Horizontal, symbol Connector_Generic:Conn_01x02
- added J12: FAN2_5V, TerminalBlock_Phoenix:TerminalBlock_Phoenix_MKDS-3-2-5.08_1x02_P5.08mm_Horizontal, symbol Connector_Generic:Conn_01x02
Connections:
- net GND: now also J11.2 (Pin_2), J12.2 (Pin_2)
- net V5: now also J11.1 (Pin_1), J12.1 (Pin_1)
- net V24 renamed +24V
Other:
- note removed: "K1 contactor: J2 low-current switch drives coil + D5 flyback. K2 bypass: Q1(2N7002 low-side)+Rg/Rgs gate+D6 flyback; MCU drives gate ~500ms after inrush via J9(CTRL). Bucks U1/U2/U3 EN=always-on(verify pullup), U2=DNP. U4/K1/K2 need real part numbers. Provisional F1(BMS)/F4(stepper)/servo-stall/7S."
- moved on the sheet: C1, C10, C2, C3, C4, C5, C6, C7, C8, C9, D1, D2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
